File: lta-logic-module/quad_led.kicad_sch (KiCad schematic)
At the start: 21 parts

Commit message: Move "like-the-art" into logic-module subproject.
Parts:
- R? (x4): value (none) -> 220R
- R? (x4): value (none) -> 5k6
- R?: value (none) -> 680R
Changed lines of the file:
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@@
     (in_bom yes) (on_board yes) (fields_autoplaced)
     (property "Reference" "R?" (id 0) (at 145.415 45.0936 90))
-    (property "Value" "" (id 1) (at 145.415 47.6305 90))
+    (property "Value" "220R" (id 1) (at 145.415 47.6305 90))
     (property "Footprint" "" (id 2) (at 145.415 49.53 0)
       (effects (font (size 1.27 1.27)) hide)
@@
       (effects (font (size 1.27 1.27)) (justify left))
     )
-    (property "Value" "" (id 1) (at 121.5136 48.0572 0)
+    (property "Value" "220R" (id 1) (at 121.5136 48.0572 0)
       (effects (font (size 1.27 1.27)) (justify left))
     )
@@
     (in_bom yes) (on_board yes) (fields_autoplaced)
     (property "Reference" "R?" (id 0) (at 170.18 46.3636 90))
-    (property "Value" "" (id 1) (at 170.18 48.9005 90))
+    (property "Value" "220R" (id 1) (at 170.18 48.9005 90))
     (property "Footprint" "" (id 2) (at 170.18 50.8 0)
       (effects (font (size 1.27 1.27)) hide)
@@
     (in_bom yes) (on_board yes) (fields_autoplaced)
     (property "Reference" "R?" (id 0) (at 64.135 102.2436 90))
-    (property "Value" "" (id 1) (at 64.135 104.7805 90))
+    (property "Value" "5k6" (id 1) (at 64.135 104.7805 90))
     (property "Footprint" "" (id 2) (at 64.135 106.68 0)
       (effects (font (size 1.27 1.27)) hide)
@@
     (in_bom yes) (on_board yes) (fields_autoplaced)
     (property "Reference" "R?" (id 0) (at 55.245 99.0686 90))
-    (property "Value" "" (id 1) (at 55.245 101.6055 90))
+    (property "Value" "5k6" (id 1) (at 55.245 101.6055 90))
     (property "Footprint" "" (id 2) (at 55.245 103.505 0)
       (effects (font (size 1.27 1.27)) hide)
@@
     (in_bom yes) (on_board yes) (fields_autoplaced)
     (property "Reference" "R?" (id 0) (at 201.295 47.6336 90))
-    (property "Value" "" (id 1) (at 201.295 50.1705 90))
+    (property "Value" "220R" (id 1) (at 201.295 50.1705 90))
     (property "Footprint" "" (id 2) (at 201.295 52.07 0)
       (effects (font (size 1.27 1.27)) hide)
@@
     (in_bom yes) (on_board yes) (fields_autoplaced)
     (property "Reference" "R?" (id 0) (at 98.425 111.7686 90))
-    (property "Value" "" (id 1) (at 98.425 114.3055 90))
+    (property "Value" "680R" (id 1) (at 98.425 114.3055 90))
     (property "Footprint" "" (id 2) (at 98.425 116.205 0)
       (effects (font (size 1.27 1.27)) hide)
@@
     (in_bom yes) (on_board yes) (fields_autoplaced)
     (property "Reference" "R?" (id 0) (at 71.755 105.4186 90))
-    (property "Value" "" (id 1) (at 71.755 107.9555 90))
+    (property "Value" "5k6" (id 1) (at 71.755 107.9555 90))
     (property "Footprint" "" (id 2) (at 71.755 109.855 0)
       (effects (font (size 1.27 1.27)) hide)
@@
     (in_bom yes) (on_board yes) (fields_autoplaced)
     (property "Reference" "R?" (id 0) (at 47.625 95.8936 90))
-    (property "Value" "" (id 1) (at 47.625 98.4305 90))
+    (property "Value" "5k6" (id 1) (at 47.625 98.4305 90))
     (property "Footprint" "" (id 2) (at 47.625 100.33 0)
       (effects (font (size 1.27 1.27)) hide)
