File: lta-logic-module/light_sensor.kicad_sch (KiCad schematic)
At the start: 9 parts, among them SW1 SW_SPST

Commit message: Switch 12-pin headers to Molex Micro-Latch c'tors.
Parts:
- JP1: value Jumper_3_Open -> (none)
- SW1: value SW_SPST -> (none)
Changed lines of the file:
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@@
       (effects (font (size 1.27 1.27)) (justify right))
     )
-    (property "Value" "SW_SPST" (id 1) (at 123.698 36.6272 90)
+    (property "Value" "" (id 1) (at 123.698 36.6272 90)
       (effects (font (size 1.27 1.27)) (justify right))
     )
@@
       (effects (font (size 1.27 1.27)) (justify left))
     )
-    (property "Value" "Jumper_3_Open" (id 1) (at 120.4209 51.2322 90)
+    (property "Value" "" (id 1) (at 120.4209 51.2322 90)
       (effects (font (size 1.27 1.27)) (justify left))
     )
