File: lta-logic-module/light_sensor.kicad_sch (KiCad schematic)
At the start: 15 parts

Commit message: Update logic module power budget from button LED measurements.
Button LEDs draw ~11mA each (98 mA total) empirically; not the ~20mA each
I initially guessed for estimating purposes.
Parts:
- D4: value (none) -> DARK_EN; footprint (none) -> LED_SMD:LED_0603_1608Metric
- JP1: value (none) -> Jumper_3_Open; footprint (none) -> Connector_PinHeader_2.54mm:PinHeader_1x03_P2.54mm_Vertical
- Q1: value (none) -> PT334-6B; footprint (none) -> Connector_PinHeader_2.54mm:PinHeader_1x02_P2.54mm_Vertical
- Q2: value (none) -> 2N3904; footprint (none) -> Package_TO_SOT_THT:TO-92_Inline
- R27, R30: value (none) -> 4K7; footprint (none) -> Resistor_SMD:R_0603_1608Metric
- R28: value (none) -> 470R; footprint (none) -> Resistor_SMD:R_0603_1608Metric
- R29: value (none) -> 220R; footprint (none) -> Resistor_SMD:R_0603_1608Metric
- R31: value (none) -> 220K; footprint (none) -> Resistor_SMD:R_0603_1608Metric
- R32: value (none) -> 120R; footprint (none) -> Resistor_SMD:R_0603_1608Metric
- RV1: value (none) -> 25K; footprint (none) -> Aaron_THT:TRIM_3362P
- SW1: value (none) -> SW_SPST; footprint (none) -> Aaron_THT:CUI-DIP-SW_DS01-254-x-01xx
- TP19, TP20: value (none) -> TestPoint_Flag; footprint (none) -> Aaron_THT:TestPoint_THTPad_1.0x1.0mm_Drill0.3mm
- TP27: value (none) -> Thief; footprint (none) -> Aaron_Pads:Pad_D1.0mm
Changed lines of the file:
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@@
       (effects (font (size 1.27 1.27)) (justify left))
     )
-    (property "Value" "" (id 1) (at 160.909 187.6302 0)
-      (effects (font (size 1.27 1.27)) (justify left))
-    )
-    (property "Footprint" "" (id 2) (at 159.385 187.325 0)
+    (property "Value" "TestPoint_Flag" (id 1) (at 160.909 187.6302 0)
+      (effects (font (size 1.27 1.27)) (justify left))
+    )
+    (property "Footprint" "Aaron_THT:TestPoint_THTPad_1.0x1.0mm_Drill0.3mm" (id 2) (at 159.385 187.325 0)
       (effects (font (size 1.27 1.27)) hide)
     )
@@
       (effects (font (size 1.27 1.27)) (justify right))
     )
-    (property "Value" "" (id 1) (at 123.698 29.6422 90)
-      (effects (font (size 1.27 1.27)) (justify right))
-    )
-    (property "Footprint" "" (id 2) (at 122.555 27.94 0)
+    (property "Value" "SW_SPST" (id 1) (at 123.698 29.6422 90)
+      (effects (font (size 1.27 1.27)) (justify right))
+    )
+    (property "Footprint" "Aaron_THT:CUI-DIP-SW_DS01-254-x-01xx" (id 2) (at 122.555 27.94 0)
       (effects (font (size 1.27 1.27)) hide)
     )
@@
     (in_bom yes) (on_board yes) (fields_autoplaced)
     (property "Reference" "R29" (id 0) (at 102.235 51.4436 90))
-    (property "Value" "" (id 1) (at 102.235 53.9805 90))
-    (property "Footprint" "" (id 2) (at 102.235 55.88 0)
+    (property "Value" "220R" (id 1) (at 102.235 53.9805 90))
+    (property "Footprint" "Resistor_SMD:R_0603_1608Metric" (id 2) (at 102.235 55.88 0)
       (effects (font (size 1.27 1.27)) hide)
     )
@@
       (effects (font (size 1.27 1.27)) (justify left))
     )
-    (property "Value" "" (id 1) (at 132.9436 62.6622 0)
-      (effects (font (size 1.27 1.27)) (justify left))
-    )
-    (property "Footprint" "" (id 2) (at 131.445 60.96 0)
+    (property "Value" "220K" (id 1) (at 132.9436 62.6622 0)
+      (effects (font (size 1.27 1.27)) (justify left))
+    )
+    (property "Footprint" "Resistor_SMD:R_0603_1608Metric" (id 2) (at 131.445 60.96 0)
       (effects (font (size 1.27 1.27)) hide)
     )
@@
       (effects (font (size 1.27 1.27)) (justify left))
     )
-    (property "Value" "" (id 1) (at 93.5736 51.8672 0)
-      (effects (font (size 1.27 1.27)) (justify left))
-    )
-    (property "Footprint" "" (id 2) (at 92.075 50.165 0)
+    (property "Value" "470R" (id 1) (at 93.5736 51.8672 0)
+      (effects (font (size 1.27 1.27)) (justify left))
+    )
+    (property "Footprint" "Resistor_SMD:R_0603_1608Metric" (id 2) (at 92.075 50.165 0)
       (effects (font (size 1.27 1.27)) hide)
     )
@@
       (effects (font (size 1.27 1.27)) (justify left))
     )
-    (property "Value" "" (id 1) (at 94.3864 69.6472 0)
-      (effects (font (size 1.27 1.27)) (justify left))
-    )
-    (property "Footprint" "" (id 2) (at 94.615 65.405 0)
+    (property "Value" "2N3904" (id 1) (at 94.3864 69.6472 0)
+      (effects (font (size 1.27 1.27)) (justify left))
+    )
+    (property "Footprint" "Package_TO_SOT_THT:TO-92_Inline" (id 2) (at 94.615 65.405 0)
       (effects (font (size 1.27 1.27)) hide)
     )
@@
       (effects (font (size 1.27 1.27)) (justify right))
     )
-    (property "Value" "" (id 1) (at 144.018 40.3737 90)
-      (effects (font (size 1.27 1.27)) (justify right))
-    )
-    (property "Footprint" "" (id 2) (at 142.24 38.735 90)
+    (property "Value" "DARK_EN" (id 1) (at 144.018 40.3737 90)
+      (effects (font (size 1.27 1.27)) (justify right))
+    )
+    (property "Footprint" "LED_SMD:LED_0603_1608Metric" (id 2) (at 142.24 38.735 90)
       (effects (font (size 1.27 1.27)) hide)
     )
@@
       (effects (font (size 1.27 1.27)) (justify left))
     )
-    (property "Value" "" (id 1) (at 120.4209 51.2322 90)
-      (effects (font (size 1.27 1.27)) (justify left))
-    )
-    (property "Footprint" "" (id 2) (at 122.555 49.53 0)
+    (property "Value" "Jumper_3_Open" (id 1) (at 120.4209 51.2322 90)
+      (effects (font (size 1.27 1.27)) (justify left))
+    )
+    (property "Footprint" "Connector_PinHeader_2.54mm:PinHeader_1x03_P2.54mm_Vertical" (id 2) (at 122.555 49.53 0)
       (effects (font (size 1.27 1.27)) hide)
     )
@@
       (effects (font (size 1.27 1.27)) (justify right))
     )
-    (property "Value" "" (id 1) (at 96.393 75.9972 0)
-      (effects (font (size 1.27 1.27)) (justify right))
-    )
-    (property "Footprint" "" (id 2) (at 90.17 74.295 0)
+    (property "Value" "Thief" (id 1) (at 96.393 75.9972 0)
+      (effects (font (size 1.27 1.27)) (justify right))
+    )
+    (property "Footprint" "Aaron_Pads:Pad_D1.0mm" (id 2) (at 90.17 74.295 0)
       (effects (font (size 1.27 1.27)) hide)
     )
@@
       (effects (font (size 1.27 1.27)) (justify left))
     )
-    (property "Value" "" (id 1) (at 75.7936 62.6622 0)
-      (effects (font (size 1.27 1.27)) (justify left))
-    )
-    (property "Footprint" "" (id 2) (at 74.295 60.96 0)
+    (property "Value" "4K7" (id 1) (at 75.7936 62.6622 0)
+      (effects (font (size 1.27 1.27)) (justify left))
+    )
+    (property "Footprint" "Resistor_SMD:R_0603_1608Metric" (id 2) (at 74.295 60.96 0)
       (effects (font (size 1.27 1.27)) hide)
     )
@@
       (effects (font (size 1.27 1.27)) (justify left))
     )
-    (property "Value" "" (id 1) (at 124.0536 41.0722 0)
-      (effects (font (size 1.27 1.27)) (justify left))
-    )
-    (property "Footprint" "" (id 2) (at 122.555 39.37 0)
+    (property "Value" "4K7" (id 1) (at 124.0536 41.0722 0)
+      (effects (font (size 1.27 1.27)) (justify left))
+    )
+    (property "Footprint" "Resistor_SMD:R_0603_1608Metric" (id 2) (at 122.555 39.37 0)
       (effects (font (size 1.27 1.27)) hide)
     )
@@
       (effects (font (size 1.27 1.27)) (justify left))
     )
-    (property "Value" "" (id 1) (at 76.6064 50.4829 0)
-      (effects (font (size 1.27 1.27)) (justify left))
-    )
-    (property "Footprint" "" (id 2) (at 76.835 46.99 0)
+    (property "Value" "PT334-6B" (id 1) (at 76.6064 50.4829 0)
+      (effects (font (size 1.27 1.27)) (justify left))
+    )
+    (property "Footprint" "Connector_PinHeader_2.54mm:PinHeader_1x02_P2.54mm_Vertical" (id 2) (at 76.835 46.99 0)
       (effects (font (size 1.27 1.27)) hide)
     )
@@
     (in_bom yes) (on_board yes) (fields_autoplaced)
     (property "Reference" "R32" (id 0) (at 135.255 29.8536 90))
-    (property "Value" "" (id 1) (at 135.255 32.3905 90))
-    (property "Footprint" "" (id 2) (at 135.255 34.29 0)
+    (property "Value" "120R" (id 1) (at 135.255 32.3905 90))
+    (property "Footprint" "Resistor_SMD:R_0603_1608Metric" (id 2) (at 135.255 34.29 0)
       (effects (font (size 1.27 1.27)) hide)
     )
@@
       (effects (font (size 1.27 1.27)) (justify left))
     )
-    (property "Value" "" (id 1) (at 161.29 192.405 0)
-      (effects (font (size 1.27 1.27)) (justify left))
-    )
-    (property "Footprint" "" (id 2) (at 159.385 192.405 0)
+    (property "Value" "TestPoint_Flag" (id 1) (at 161.29 192.405 0)
+      (effects (font (size 1.27 1.27)) (justify left))
+    )
+    (property "Footprint" "Aaron_THT:TestPoint_THTPad_1.0x1.0mm_Drill0.3mm" (id 2) (at 159.385 192.405 0)
       (effects (font (size 1.27 1.27)) hide)
     )
@@
       (effects (font (size 1.27 1.27)) (justify right))
     )
-    (property "Value" "" (id 1) (at 93.726 41.7072 0)
-      (effects (font (size 1.27 1.27)) (justify right))
-    )
-    (property "Footprint" "" (id 2) (at 92.075 40.005 0)
-      (effects (font (size 1.27 1.27)) hide)
-    )
+    (property "Value" "25K" (id 1) (at 93.726 41.7072 0)
+      (effects (font (size 1.27 1.27)) (justify right))
+    )
+    (property "Footprint" "Aaron_THT:TRIM_3362P" (id 2) (at 92.075 40.005 0)
+      (effects (font (size 1.27 1.27)) hide)
+    )
