File: lta-power-module/lta-power-module.kicad_pcb (KiCad board)
At the start: 2 copper layers, 289.9 x 205.9 mm, 306 parts, among them J1 Molex-MicroLatch-53253-0270, J10 Conn_01x01, J100 Conn_01x01, J101 Conn_01x01, J102 Conn_01x01, J103 Conn_01x01, J104 Conn_01x01, J105 Conn_01x01, J106 Conn_01x01, J107 Conn_01x01, J108 Conn_01x01, J109 Conn_01x01, J11 Conn_01x01, J110 Conn_01x01, J112 Conn_01x01, J113 Conn_01x01, J114 Conn_01x01, J115 Conn_01x01, J116 Conn_01x01, J117 Conn_01x01, J118 Conn_01x01, J119 Conn_01x01, J12 Conn_01x01, J120 Conn_01x01, J121 Conn_01x01, J122 Conn_01x01, J123 Conn_01x01, J124 Conn_01x01, J126 Conn_01x01, J127 Conn_01x01, J128 Conn_01x01, J129 Conn_01x01, J13 Conn_01x01, J130 Conn_01x01, J131 Conn_01x01, J132 Conn_01x01, J133 Conn_01x01, J134 Conn_01x01, J135 Conn_01x01, J136 Conn_01x01, J137 Conn_01x01, J138 Conn_01x01, J14 Conn_01x01, J140 Conn_01x01, J141 Conn_01x01, J142 Conn_01x01, J143 Conn_01x01, J144 Conn_01x01, J145 Conn_01x01, J146 Conn_01x01, J147 Conn_01x01, J148 Conn_01x01, J149 Conn_01x01, J15 Conn_01x01, J150 Conn_01x01, J151 Conn_01x01, J152 Conn_01x01, J153 Conn_01x01, J154 Conn_01x01, J155 Conn_01x01, J156 Conn_01x01, J157 Conn_01x01, J158 Conn_01x01, J159 Conn_01x01, J16 Conn_01x01, J160 Conn_01x01, J161 Conn_01x01, J162 Conn_01x01, J164 Conn_01x01, J165 Conn_01x01, J166 Conn_01x01, J167 Conn_01x01, J168 Conn_01x01, J169 Conn_01x01, J17 Conn_01x01, J170 Conn_01x01, J171 Conn_01x01, J172 Conn_01x01, J173 Conn_01x01, J174 Conn_01x01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

Commit message: Add protoboard.
Parts:
- removed J136, J150, J174, J188, J202, J212, J32, J84: Conn_01x01, Aaron_Pads:1.6mm_PTH_No_Silk
- removed J137, J151, J175, J189, J203, J213, J33, J85: Conn_01x01, Aaron_Pads:1mm_PTH_No_Silk
- J107, J121, J135, J149, J159, J17, J173, J187, J201, J211, J31, J45, J59, J69, J83, J97: footprint Aaron_Pads:1.6mm_PTH_No_Silk -> Aaron_Pads:1mm_PTH_No_Silk
- moved J6 273.0 mm to (139.7, 40.6), turned to 90 degrees
- moved J162 264.0 mm to (139.7, 33.0), turned to 90 degrees
- moved J50 263.1 mm to (142.2, 33.0), turned to 90 degrees
- moved J228 261.2 mm to (142.2, 35.5), turned to 90 degrees
- moved J72 260.5 mm to (139.7, 35.5), turned to 90 degrees
- moved J48 260.3 mm to (139.7, 43.1), turned to 90 degrees
- moved J112 258.4 mm to (142.2, 38.1), turned to 90 degrees
- moved J176 258.3 mm to (139.7, 45.7), turned to 90 degrees
- moved J126 258.2 mm to (142.2, 45.7), turned to 90 degrees
- moved J80 257.3 mm to (152.4, 35.5)
- moved J138 256.9 mm to (139.7, 38.1), turned to 90 degrees
- moved J82 256.4 mm to (154.9, 35.5)
- moved J16 255.7 mm to (149.9, 33.0)
- moved J88 255.0 mm to (142.2, 40.6), turned to 90 degrees
- moved J148 254.9 mm to (147.3, 58.3)
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Routing:
- net VDD: track 454.9 -> 553.8 mm, vias 8 -> 9
- net VCC0: track 397.2 -> 468.8 mm
- net Net-(J128-Pad1): track 0.00 -> 7.65 mm
- net Net-(J10-Pad1): track 0.00 -> 7.64 mm
- net Net-(J24-Pad1): track 0.00 -> 7.62 mm
- net Net-(J14-Pad1): track 0.00 -> 7.62 mm
- net Net-(J80-Pad1): track 0.00 -> 7.61 mm
- net Net-(J94-Pad1): track 0.00 -> 7.60 mm
- net Net-(J38-Pad1): track 0.00 -> 7.59 mm
- net Net-(J118-Pad1): track 0.00 -> 7.59 mm
- net Net-(J62-Pad1): track 0.00 -> 7.57 mm
- net Net-(J198-Pad1): track 0.00 -> 7.57 mm
- net Net-(J90-Pad1): track 0.00 -> 7.56 mm
- net Net-(J184-Pad1): track 0.00 -> 7.56 mm
- net Net-(J52-Pad1): track 0.00 -> 7.55 mm
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Other:
- board text added: "+12"
- board text added: "+5"
- board text added: "BANK 0 INPUT SIGNALS: LED0..LED7"
- board text added: "BANK 1 INPUT SIGNALS: LED8..LED15"
- board text added: "GND"
- board text added: "LED0"
- board text added: "LED1"
- board text added: "LED10"
- board text added: "LED11"
- board text added: "LED12"
- board text added: "LED13"
- board text added: "LED14"
- board text added: "LED15"
- board text added: "LED2"
- board text added: "LED3"
- board text added: "LED4"
- board text added: "LED5"
- board text added: "LED6"
- board text added: "LED7"
- board text added: "LED8"
- board text added: "LED9"
- board text added: "[OUT0]"
- board text added: "[OUT15]"
- board text removed: "BANK 0 SIGNALS: LED0..LED7"
- board text removed: "BANK 1 SIGNALS: LED8..LED15"
- board text removed: "[Q16]"
- board text removed: "[Q1]"

Commit message: Work on border.
* Add perimeter edge cut to fit WH-22 polycase.
* Add M5 mounting holes in temp locations on PCB.
* Lay out and lock left-edge M5 mounting holes.
Parts:
- added H1: MountingHole_Pad, MountingHole:MountingHole_5.3mm_M5_ISO7380_Pad, F.Cu at (337.8, 68.6)
- added H10: MountingHole_Pad, MountingHole:MountingHole_5.3mm_M5_ISO7380_Pad, F.Cu at (287.0, 27.9)
- added H11: MountingHole_Pad, MountingHole:MountingHole_5.3mm_M5_ISO7380_Pad, F.Cu at (31.2, 193.7)
- added H12: MountingHole_Pad, MountingHole:MountingHole_5.3mm_M5_ISO7380_Pad, F.Cu at (104.1, 30.5)
- added H2: MountingHole_Pad, MountingHole:MountingHole_5.3mm_M5_ISO7380_Pad, F.Cu at (337.8, 190.5)
- added H3: MountingHole_Pad, MountingHole:MountingHole_5.3mm_M5_ISO7380_Pad, F.Cu at (154.9, 27.9)
- added H4: MountingHole_Pad, MountingHole:MountingHole_5.3mm_M5_ISO7380_Pad, F.Cu at (147.3, 236.2)
- added H5: MountingHole_Pad, MountingHole:MountingHole_5.3mm_M5_ISO7380_Pad, F.Cu at (228.6, 236.2)
- added H6: MountingHole_Pad, MountingHole:MountingHole_5.3mm_M5_ISO7380_Pad, F.Cu at (31.2, 68.7)
- added H7: MountingHole_Pad, MountingHole:MountingHole_5.3mm_M5_ISO7380_Pad, F.Cu at (96.5, 236.2)
- added H8: MountingHole_Pad, MountingHole:MountingHole_5.3mm_M5_ISO7380_Pad, F.Cu at (292.1, 236.2)
- added H9: MountingHole_Pad, MountingHole:MountingHole_5.3mm_M5_ISO7380_Pad, F.Cu at (228.6, 27.9)
- moved R25 20.2 mm to (146.2, 166.2)
- moved J101 20.2 mm to (185.7, 72.6)
- moved J109 20.2 mm to (156.2, 92.5)
- moved J116 20.2 mm to (185.7, 77.6)
- moved J123 20.2 mm to (156.2, 87.4)
- moved J13 20.2 mm to (188.2, 47.3)
- moved J138 20.2 mm to (157.7, 47.3)
- moved J176 20.2 mm to (157.7, 54.9)
- moved J182 20.2 mm to (185.7, 80.2)
- moved J190 20.2 mm to (157.7, 80.2)
- moved J197 20.2 mm to (185.7, 75.1)
- moved J20 20.2 mm to (157.7, 57.4)
- moved J214 20.2 mm to (157.7, 59.9)
- moved J218 20.2 mm to (157.7, 77.6)
- moved J222 20.2 mm to (157.7, 72.6)
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Other:
- board size 289.9 x 205.9 mm -> 310 x 210 mm

Commit message: Lay out all mounting holes.
* All DRC checks passing.
* Fix footprint silkscreen conflicts.
* Fix ext. regulator module symbol.
Parts:
- D1, D2, D4: footprint LED_THT:LED_D5.0mm -> Aaron_THT:LED_D5.0mm_SilkFix
- moved H8 25.1 mm to (267.8, 230.2)
- moved H10 19.7 mm to (267.8, 32.2)
- moved J4 19.3 mm to (232.6, 39.1)
- moved H3 12.9 mm to (142.8, 32.2)
- moved H5 12.4 mm to (217.8, 230.2)
- moved H9 11.6 mm to (217.8, 32.2)
- moved H12 11.5 mm to (92.8, 32.2)
- moved H2 9.19 mm to (329.2, 193.7)
- moved H1 8.61 mm to (329.2, 68.7)
- moved H4 7.53 mm to (142.8, 230.2)
- moved H7 7.07 mm to (92.8, 230.2)
- moved J3 6.67 mm to (106.9, 38.4)
Routing:
- net /Signal Input Processing/s9: track 140.2 -> 151.5 mm
- net /Signal Input Processing/s8: track 131.9 -> 143.1 mm
- net /Signal Input Processing/s10: track 130.2 -> 139.3 mm
- net /Signal Input Processing/s11: track 129.0 -> 137.6 mm
- net /Signal Input Processing/s12: track 143.0 -> 139.3 mm
- net /Signal Input Processing/s13: track 139.8 -> 136.4 mm
- net /Signal Input Processing/s7: track 140.0 -> 143.0 mm
- net /Signal Input Processing/s4: track 138.1 -> 141.0 mm
- net /Signal Input Processing/s3: track 132.8 -> 135.8 mm
- net /Signal Input Processing/s1: track 131.6 -> 134.6 mm
- net /Signal Input Processing/s6: track 139.7 -> 142.6 mm
- net /Signal Input Processing/s5: track 139.6 -> 142.5 mm
- net /Signal Input Processing/s2: track 136.4 -> 139.4 mm
- net /Signal Input Processing/s0: track 127.0 -> 130.0 mm
- net /Signal Input Processing/s14: track 134.2 -> 133.0 mm
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
Commit message: NPTHs and test points.
* Added NPTH defs to `User.Eco1` layer in footprints.
* Renamed `User.Eco1` to `Mechanical` in PCB layout.
* Duplicated `Edge Cuts` onto `Mechanical` layer.
  *Use `Mechanical` as `.GKO` layer, not `Edge Cuts`!*
* Added test points for key signals.
Parts:
- added TP10: TestPoint_Flag, Aaron_THT:TestPoint_THTPad_1.0x1.0mm_Drill0.3mm, F.Cu at (174.0, 219.4)
- added TP11: TestPoint_Flag, Aaron_THT:TestPoint_THTPad_1.0x1.0mm_Drill0.3mm, F.Cu at (88.4, 40.9)
- added TP12: TestPoint_Flag, Aaron_THT:TestPoint_THTPad_1.0x1.0mm_Drill0.3mm, F.Cu at (267.2, 41.4)
- added TP13: TestPoint_Flag, Aaron_THT:TestPoint_THTPad_1.0x1.0mm_Drill0.3mm, F.Cu at (261.6, 41.4)
- added TP14: TestPoint_Flag, Aaron_THT:TestPoint_THTPad_1.0x1.0mm_Drill0.3mm, F.Cu at (93.7, 40.9)
- added TP15: TestPoint_Flag, Aaron_THT:TestPoint_THTPad_1.0x1.0mm_Drill0.3mm, F.Cu at (168.7, 219.5)
- added TP16: TestPoint_Flag, Aaron_THT:TestPoint_THTPad_1.0x1.0mm_Drill0.3mm, F.Cu at (178.8, 219.5)
- added TP8: TestPoint_Flag, Aaron_THT:TestPoint_THTPad_1.0x1.0mm_Drill0.3mm, F.Cu at (158.4, 219.5)
- added TP9: TestPoint_Flag, Aaron_THT:TestPoint_THTPad_1.0x1.0mm_Drill0.3mm, F.Cu at (196.5, 219.5)
- moved J4 3.05 mm to (232.6, 36.1)
- moved J3 2.33 mm to (106.9, 36.1)
Routing:
- net /Signal Input Processing/s0: track 130.0 -> 148.1 mm
- net /Signal Input Processing/s15: track 130.5 -> 141.0 mm
- net /Signal Input Processing/out8: track 35.7 -> 41.8 mm
- net /Signal Input Processing/out4: track 40.4 -> 46.5 mm
- net /Signal Input Processing/out0: track 57.7 -> 63.8 mm
- net /Signal Input Processing/out15: track 56.4 -> 62.4 mm
- net /Signal Input Processing/s8: track 143.1 -> 146.2 mm
- net /Signal Input Processing/s9: track 151.5 -> 154.5 mm
- net /Signal Input Processing/s14: track 133.0 -> 136.0 mm
- net /Signal Input Processing/s13: track 136.4 -> 139.4 mm
- net /Signal Input Processing/s12: track 139.3 -> 142.3 mm
- net /Signal Input Processing/s10: track 139.3 -> 142.3 mm
- net /Signal Input Processing/s11: track 137.6 -> 140.6 mm
- net /Signal Input Processing/s2: track 139.4 -> 141.7 mm
- net /Signal Input Processing/s6: track 142.6 -> 144.9 mm
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Other:
- board text added: "12V0"
- board text added: "OUT4"
- board text added: "OUT8"
- board text added: "s0"
- board text added: "s15"
- board text removed: "+12"
- board text removed: "+5"
