File: lta-power-module/lta-power-module.kicad_pcb (KiCad board)
At the start: 2 copper layers, 310 x 210 mm, 311 parts, among them J1 Molex-MicroLatch-53253-0270, J10 Conn_01x01, J100 Conn_01x01, J101 Conn_01x01, J102 Conn_01x01, J103 Conn_01x01, J104 Conn_01x01, J105 Conn_01x01, J106 Conn_01x01, J107 Conn_01x01, J108 Conn_01x01, J109 Conn_01x01, J11 Conn_01x01, J110 Conn_01x01, J112 Conn_01x01, J113 Conn_01x01, J114 Conn_01x01, J115 Conn_01x01, J116 Conn_01x01, J117 Conn_01x01, J118 Conn_01x01, J119 Conn_01x01, J12 Conn_01x01, J120 Conn_01x01, J121 Conn_01x01, J122 Conn_01x01, J123 Conn_01x01, J124 Conn_01x01, J126 Conn_01x01, J127 Conn_01x01, J128 Conn_01x01, J129 Conn_01x01, J13 Conn_01x01, J130 Conn_01x01, J131 Conn_01x01, J132 Conn_01x01, J133 Conn_01x01, J134 Conn_01x01, J135 Conn_01x01, J138 Conn_01x01, J14 Conn_01x01, J140 Conn_01x01, J141 Conn_01x01, J142 Conn_01x01, J143 Conn_01x01, J144 Conn_01x01, J145 Conn_01x01, J146 Conn_01x01, J147 Conn_01x01, J148 Conn_01x01, J149 Conn_01x01, J15 Conn_01x01, J152 Conn_01x01, J153 Conn_01x01, J154 Conn_01x01, J155 Conn_01x01, J156 Conn_01x01, J157 Conn_01x01, J158 Conn_01x01, J159 Conn_01x01, J16 Conn_01x01, J160 Conn_01x01, J161 Conn_01x01, J162 Conn_01x01, J164 Conn_01x01, J165 Conn_01x01, J166 Conn_01x01, J167 Conn_01x01, J168 Conn_01x01, J169 Conn_01x01, J17 Conn_01x01, J170 Conn_01x01, J171 Conn_01x01, J172 Conn_01x01, J173 Conn_01x01, J176 Conn_01x01, J178 Conn_01x01, J179 Conn_01x01, J18 Conn_01x01, J180 Conn_01x01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

Commit message: Update module footprints to be more accurate.
Routing:
- net GND: vias 48 -> 52

Commit message: Open solder masks up around mounting holes.
Routing:
- net GND: vias 52 -> 54
Other:
- rule pad_to_mask_clearance: 0 -> 0.05
- board text added: "TODO: NPTH holes without copper pad should ALWAYS have a soldermask clearance pad"
- board text added: "YOU DON'T HAVE TO LIKE ALL THE ART! POWER MODULE - V${REV}"
- board text removed: "YOU DON'T HAVE TO LIKE ALL THE ART! POWER MODULE - V1.0"

Commit message: Switched to plated through-holes for all mounting.
Ready for release to manufacturing.
Routing:
- net VDD: track 553.8 -> 555.1 mm
- net VCC0: track 468.3 -> 467.1 mm
- net GND: vias 54 -> 60
Other:
- board text added: "PWR"
- board text removed: "TODO: NPTH holes without copper pad should ALWAYS have a soldermask clearance pad"
