File: lta-power-module/signals_in.kicad_sch (KiCad schematic)
At the start: 55 parts

Commit message: Considerably more work on power module PCB.
* Slight reorganization of layout.
* Routed all traces.
Parts:
- R10, R11, R24, R25, R26, R27, R35, R36, R39, R40, R46, R47, R53, R54, R8, R9: Comment 22K THT resistor; +/-5%; 1/8W -> 2K2 THT resistor; +/-5%; 1/8W; MPN CF18JT22K0 -> CF18JT2K20
- R28, R29, R34, R38, R48, R55, R6, R7: Comment 470R THT resistor; +/-5%; 1/8W -> 220R THT resistor; +/-5%; 1/8W; MPN CF18JT470R0 -> CF18JT220R

Commit message: Add protoboard.
Parts:
- C10, C3, C4, C5, C6, C7, C8, C9: SPN (none) -> 399-C315C105K3R5TA7303CT-ND; Supplier (none) -> DigiKey
- J3, J4: SPN (none) -> WM24308-ND; Supplier (none) -> DigiKey
- J5: MANUFACTURER (none) -> TE Connectivity AMP Connectors; MPN (none) -> 5-146858-1; SPN (none) -> A105469CT-ND; Supplier (none) -> DigiKey
- R10, R11, R24, R25, R26, R27, R35, R36, R39, R40, R46, R47, R53, R54, R8, R9: SPN (none) -> CF18JT2K20CT-ND; Supplier (none) -> DigiKey
- R12, R13, R14, R15, R20, R21, R22, R23, R37, R41, R42, R43, R44, R45, R51, R52: SPN (none) -> CF18JT33R0CT-ND; Supplier (none) -> DigiKey
- R28, R29, R34, R38, R48, R55, R6, R7: SPN (none) -> CF18JT220RCT-ND; Supplier (none) -> DigiKey
- U6, U7, U8, U9: SPN (none) -> 296-34130-5-ND; Supplier (none) -> DigiKey

Commit message: Work on border.
* Add perimeter edge cut to fit WH-22 polycase.
* Add M5 mounting holes in temp locations on PCB.
* Lay out and lock left-edge M5 mounting holes.
Parts:
- J3, J4: Comment (none) -> 12-pin signal connector
Changed lines of the file:
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@@
+      (effects (font (size 1.27 1.27)) hide)
+    )
+    (property "Comment" "12-pin signal connector" (id 8) (at 41.91 65.405 0)
       (effects (font (size 1.27 1.27)) hide)
     )
@@
       (effects (font (size 1.27 1.27)) hide)
     )
+    (property "Comment" "12-pin signal connector" (id 8) (at 41.91 109.22 0)
+      (effects (font (size 1.27 1.27)) hide)
+    )

Commit message: NPTHs and test points.
* Added NPTH defs to `User.Eco1` layer in footprints.
* Renamed `User.Eco1` to `Mechanical` in PCB layout.
* Duplicated `Edge Cuts` onto `Mechanical` layer.
  *Use `Mechanical` as `.GKO` layer, not `Edge Cuts`!*
* Added test points for key signals.
Parts:
- added TP13, TP14, TP15, TP16, TP8, TP9: TestPoint_Flag, Aaron_THT:TestPoint_THTPad_1.0x1.0mm_Drill0.3mm, symbol Connector:TestPoint_Flag
Connections:
- net out0: now also TP8.1
- net out15: now also TP9.1
- net out4: now also TP15.1
- net out8: now also TP16.1
- net s0: now also TP14.1
- net s15: now also TP13.1
Changed lines of the file:
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@@
   (junction (at 163.195 24.13) (diameter 0) (color 0 0 0 0)
   )
+  (junction (at 264.16 107.315) (diameter 0) (color 0 0 0 0)
+  )
   (junction (at 205.105 69.85) (diameter 0) (color 0 0 0 0)
   )
@@
   )
   (junction (at 118.11 90.17) (diameter 0) (color 0 0 0 0)
+  )
+  (junction (at 264.16 69.215) (diameter 0) (color 0 0 0 0)
   )
   (junction (at 118.11 180.34) (diameter 0) (color 0 0 0 0)
@@
     (stroke (width 0) (type default) (color 0 0 0 0))
   )
-  (wire (pts (xy 41.91 67.945) (xy 45.72 67.945))
+  (wire (pts (xy 41.91 67.945) (xy 54.61 67.945))
     (stroke (width 0) (type default) (color 0 0 0 0))
   )
@@
     (stroke (width 0) (type default) (color 0 0 0 0))
   )
+  (wire (pts (xy 264.16 107.315) (xy 264.16 114.935))
+    (stroke (width 0) (type default) (color 0 0 0 0))
+  )
   (wire (pts (xy 93.98 180.34) (xy 100.33 180.34))
     (stroke (width 0) (type default) (color 0 0 0 0))
@@
     (stroke (width 0) (type default) (color 0 0 0 0))
   )
+  (wire (pts (xy 251.46 79.375) (xy 264.16 79.375))
+    (stroke (width 0) (type default) (color 0 0 0 0))
+  )
   (wire (pts (xy 100.33 165.735) (xy 100.33 180.34))
     (stroke (width 0) (type default) (color 0 0 0 0))
@@
     (stroke (width 0) (type default) (color 0 0 0 0))
   )
+  (wire (pts (xy 45.72 142.24) (xy 50.8 142.24))
+    (stroke (width 0) (type default) (color 0 0 0 0))
+  )
   (wire (pts (xy 93.98 90.17) (xy 100.33 90.17))
     (stroke (width 0) (type default) (color 0 0 0 0))
   )
+  (wire (pts (xy 251.46 73.025) (xy 251.46 79.375))
+    (stroke (width 0) (type default) (color 0 0 0 0))
+  )
   (wire (pts (xy 203.835 161.29) (xy 203.835 165.1))
     (stroke (width 0) (type default) (color 0 0 0 0))
@@
     (stroke (width 0) (type default) (color 0 0 0 0))
   )
+  (wire (pts (xy 264.16 63.5) (xy 264.16 69.215))
+    (stroke (width 0) (type default) (color 0 0 0 0))
+  )
   (wire (pts (xy 118.11 90.17) (xy 120.015 90.17))
     (stroke (width 0) (type default) (color 0 0 0 0))
@@
     (stroke (width 0) (type default) (color 0 0 0 0))
   )
-  (wire (pts (xy 258.445 89.535) (xy 264.16 89.535))
+  (wire (pts (xy 251.46 89.535) (xy 264.16 89.535))
     (stroke (width 0) (type default) (color 0 0 0 0))
   )
@@
     (stroke (width 0) (type default) (color 0 0 0 0))
   )
-  (wire (pts (xy 258.445 79.375) (xy 264.16 79.375))
-    (stroke (width 0) (type default) (color 0 0 0 0))
-  )
   (wire (pts (xy 186.055 139.065) (xy 190.5 139.065))
     (stroke (width 0) (type default) (color 0 0 0 0))
@@
     (stroke (width 0) (type default) (color 0 0 0 0))
   )
+  (wire (pts (xy 45.72 137.16) (xy 45.72 142.24))
+    (stroke (width 0) (type default) (color 0 0 0 0))
+  )
   (wire (pts (xy 258.445 107.315) (xy 264.16 107.315))
     (stroke (width 0) (type default) (color 0 0 0 0))
@@
     (stroke (width 0) (type default) (color 0 0 0 0))
   )
+  (wire (pts (xy 251.46 86.995) (xy 251.46 89.535))
+    (stroke (width 0) (type default) (color 0 0 0 0))
+  )
   (wire (pts (xy 82.55 163.195) (xy 82.55 167.005))
     (stroke (width 0) (type default) (color 0 0 0 0))
@@
     (stroke (width 0) (type default) (color 0 0 0 0))
   )
+  (wire (pts (xy 54.61 67.945) (xy 54.61 65.405))
+    (stroke (width 0) (type default) (color 0 0 0 0))
+  )
   (wire (pts (xy 125.095 173.355) (xy 131.445 173.355))
     (stroke (width 0) (type default) (color 0 0 0 0))
@@
     (stroke (width 0) (type default) (color 0 0 0 0))
   )
-  (text "16x connections\nto onboard FET drivers" (at 261.62 61.595 0)
+  (text "16x connections\nto onboard FET drivers" (at 279.4 98.044 90)
     (effects (font (size 1.27 1.27)) (justify left bottom))
   )
@@
   )
   (symbol (lib_id "Connector_Generic:Conn_01x16") (at 269.24 86.995 0) (unit 1)
-    (in_bom yes) (on_board yes) (fields_autoplaced)
+    (in_bom yes) (on_board yes)
     (property "Reference" "J5" (id 0) (at 271.272 87.4303 0)
       (effects (font (size 1.27 1.27)) (justify left))
     )
-    (property "Value" "" (id 1) (at 271.272 89.9672 0)
+    (property "Value" "" (id 1) (at 272.542 82.804 90)
       (effects (font (size 1.27 1.27)) (justify left))
     )
@@
     (pin "1")
   )
+  (symbol (lib_id "Connector:TestPoint_Flag") (at 54.61 65.405 0) (unit 1)
+    (in_bom no) (on_board yes) (fields_autoplaced)
+    (property "Reference" "TP14" (id 0) (at 61.214 63.1733 0)
+      (effects (font (size 1.27 1.27)) (justify left))
+    )
+    (property "Value" "TestPoint_Flag" (id 1) (at 61.214 65.7102 0)
+      (effects (font (size 1.27 1.27)) (justify left))
+    )
+    (property "Footprint" "Aaron_THT:TestPoint_THTPad_1.0x1.0mm_Drill0.3mm" (id 2) (at 59.69 65.405 0)
+      (effects (font (size 1.27 1.27)) hide)
+    )
+    (property "Datasheet" "~" (id 3) (at 59.69 65.405 0)
+      (effects (font (size 1.27 1.27)) hide)
+    )
+    (pin "1")
+  )
   (symbol (lib_id "Device:R_Small") (at 214.63 63.5 90) (unit 1)
     (in_bom yes) (on_board yes)
@@
     (pin "1")
   )
+  (symbol (lib_id "Connector:TestPoint_Flag") (at 264.16 114.935 0) (unit 1)
+    (in_bom no) (on_board yes) (fields_autoplaced)
+    (property "Reference" "TP9" (id 0) (at 270.764 112.7033 0)
+      (effects (font (size 1.27 1.27)) (justify left))
+    )
+    (property "Value" "TestPoint_Flag" (id 1) (at 270.764 115.2402 0)
+      (effects (font (size 1.27 1.27)) (justify left))
+    )
+    (property "Footprint" "Aaron_THT:TestPoint_THTPad_1.0x1.0mm_Drill0.3mm" (id 2) (at 269.24 114.935 0)
+      (effects (font (size 1.27 1.27)) hide)
+    )
+    (property "Datasheet" "~" (id 3) (at 269.24 114.935 0)
+      (effects (font (size 1.27 1.27)) hide)
+    )
+    (pin "1")
+  )
   (symbol (lib_id "Device:R_Small") (at 125.095 167.005 90) (unit 1)
     (in_bom yes) (on_board yes)
@@
     (pin "1")
   )
+  (symbol (lib_id "Connector:TestPoint_Flag") (at 251.46 86.995 0) (mirror y) (unit 1)
+    (in_bom no) (on_board yes)
+    (property "Reference" "TP16" (id 0) (at 234.95 85.09 0)
+      (effects (font (size 1.27 1.27)) (justify right))
+    )
+    (property "Value" "TestPoint_Flag" (id 1) (at 234.95 87.6269 0)
+      (effects (font (size 1.27 1.27)) (justify right))
+    )
+    (property "Footprint" "Aaron_THT:TestPoint_THTPad_1.0x1.0mm_Drill0.3mm" (id 2) (at 246.38 86.995 0)
+      (effects (font (size 1.27 1.27)) hide)
+    )
+    (property "Datasheet" "~" (id 3) (at 246.38 86.995 0)
+      (effects (font (size 1.27 1.27)) hide)
+    )
+    (pin "1")
+  )
   (symbol (lib_id "Device:R_Small") (at 125.095 76.835 90) (unit 1)
     (in_bom yes) (on_board yes)
@@
     (pin "1")
     (pin "2")
+  )
+  (symbol (lib_id "Connector:TestPoint_Flag") (at 251.46 73.025 0) (mirror y) (unit 1)
+    (in_bom no) (on_board yes)
+    (property "Reference" "TP15" (id 0) (at 234.95 71.12 0)
+      (effects (font (size 1.27 1.27)) (justify right))
+    )
+    (property "Value" "TestPoint_Flag" (id 1) (at 234.95 73.6569 0)
+      (effects (font (size 1.27 1.27)) (justify right))
+    )
+    (property "Footprint" "Aaron_THT:TestPoint_THTPad_1.0x1.0mm_Drill0.3mm" (id 2) (at 246.38 73.025 0)
+      (effects (font (size 1.27 1.27)) hide)
+    )
+    (property "Datasheet" "~" (id 3) (at 246.38 73.025 0)
+      (effects (font (size 1.27 1.27)) hide)
+    )
+    (pin "1")
   )
   (symbol (lib_id "Device:R_Small") (at 226.06 145.415 270) (mirror x) (unit 1)
@@
     (pin "2")
   )
+  (symbol (lib_id "Connector:TestPoint_Flag") (at 264.16 63.5 0) (unit 1)
+    (in_bom no) (on_board yes) (fields_autoplaced)
+    (property "Reference" "TP8" (id 0) (at 270.764 61.2683 0)
+      (effects (font (size 1.27 1.27)) (justify left))
+    )
+    (property "Value" "TestPoint_Flag" (id 1) (at 270.764 63.8052 0)
+      (effects (font (size 1.27 1.27)) (justify left))
+    )
+    (property "Footprint" "Aaron_THT:TestPoint_THTPad_1.0x1.0mm_Drill0.3mm" (id 2) (at 269.24 63.5 0)
+      (effects (font (size 1.27 1.27)) hide)
+    )
+    (property "Datasheet" "~" (id 3) (at 269.24 63.5 0)
+      (effects (font (size 1.27 1.27)) hide)
+    )
+    (pin "1")
+  )
   (symbol (lib_id "power:GND") (at 135.255 42.545 0) (unit 1)
     (in_bom yes) (on_board yes) (fields_autoplaced)
@@
       (effects (font (size 1.27 1.27)) hide)
     )
+    (pin "1")
+  )
+  (symbol (lib_id "Connector:TestPoint_Flag") (at 50.8 142.24 0) (unit 1)
+    (in_bom no) (on_board yes) (fields_autoplaced)
+    (property "Reference" "TP13" (id 0) (at 57.404 140.0083 0)
+      (effects (font (size 1.27 1.27)) (justify left))
+    )
+    (property "Value" "TestPoint_Flag" (id 1) (at 57.404 142.5452 0)
+      (effects (font (size 1.27 1.27)) (justify left))
+    )
+    (property "Footprint" "Aaron_THT:TestPoint_THTPad_1.0x1.0mm_Drill0.3mm" (id 2) (at 55.88 142.24 0)
+      (effects (font (size 1.27 1.27)) hide)
+    )
+    (property "Datasheet" "~" (id 3) (at 55.88 142.24 0)
+      (effects (font (size 1.27 1.27)) hide)
+    )

Commit message: Update module footprints to be more accurate.
Parts:
- C10, C3, C4, C5, C6, C7, C8, C9: value (none) -> 1u; footprint (none) -> Capacitor_THT:C_Disc_D3.8mm_W2.6mm_P2.50mm
- J3, J4: value (none) -> Molex-MicroLatch-53253-1270; footprint (none) -> Aaron_THT:Molex-MicroLatch-53253-1270
- J5: value (none) -> Conn_01x16; footprint (none) -> Connector_PinHeader_2.54mm:PinHeader_1x16_P2.54mm_Vertical
- R10, R11, R24, R25, R26, R27, R35, R36, R39, R40, R46, R47, R53, R54, R8, R9: value (none) -> 2K2; footprint (none) -> Resistor_THT:R_Axial_DIN0204_L3.6mm_D1.6mm_P5.08mm_Horizontal
- R12, R13, R14, R15, R20, R21, R22, R23, R37, R41, R42, R43, R44, R45, R51, R52: value (none) -> 33R; footprint (none) -> Resistor_THT:R_Axial_DIN0204_L3.6mm_D1.6mm_P5.08mm_Horizontal
- R28, R29, R34, R38, R48, R55, R6, R7: value (none) -> 220R; footprint (none) -> Resistor_THT:R_Axial_DIN0204_L3.6mm_D1.6mm_P5.08mm_Horizontal
- U6, U7, U8, U9: value (none) -> SN75374N; footprint (none) -> Aaron_TI_Parts:TI_N_R-PDIP-T16
