File: mosfet-chip/mosfet-chip.kicad_sch (KiCad schematic)
At the start: 10 parts, among them J1 Conn_01x02, J2 Screw_Terminal_01x02, J3 Screw_Terminal_01x02, Q1 ${FET_PART}

Commit message: Update board for D4M.
* Fix layout violation: Move SMT components 2.5mm+ from edge.
* Update MPN/SPNs for resistors to use correct JLC basic library parts.
Parts:
- J1: JLCPCB_PN (none) -> DNP
- R1: JLCPCB_PN C105588 -> C22775; MANUFACTURER YAEGO -> UNI-ROYAL; MPN RC0603FR-07100RL -> 0603WAF1000T5E
- R2: JLCPCB_PN C25197 -> C25804; MPN 0603WAF510KT5E -> 0603WAF1002T5E
- R3: JLCPCB_PN C108078 -> C22978; MANUFACTURER YAEGO -> UNI-ROYAL; MPN RC0603FR-073K3L -> 0603WAF3301T5E
Changed lines of the file:
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@@
+      (effects (font (size 1.27 1.27)) hide)
+    )
+    (property "JLCPCB_PN" "DNP" (id 8) (at 32.385 71.12 0)
       (effects (font (size 1.27 1.27)) hide)
     )
@@
       (effects (font (size 1.27 1.27)) hide)
     )
-    (property "MPN" "0603WAF510KT5E" (id 4) (at 53.975 74.93 0)
+    (property "MPN" "0603WAF1002T5E" (id 4) (at 53.975 74.93 0)
       (effects (font (size 1.27 1.27)) hide)
     )
@@
       (effects (font (size 1.27 1.27)) hide)
     )
-    (property "JLCPCB_PN" "C25197" (id 8) (at 53.975 74.93 0)
+    (property "JLCPCB_PN" "C25804" (id 8) (at 53.975 74.93 0)
       (effects (font (size 1.27 1.27)) hide)
     )
@@
       (effects (font (size 1.27 1.27)) hide)
     )
-    (property "MPN" "RC0603FR-07100RL" (id 4) (at 49.53 71.12 90)
+    (property "MPN" "0603WAF1000T5E" (id 4) (at 49.53 71.12 90)
       (effects (font (size 1.27 1.27)) hide)
     )
@@
       (effects (font (size 1.27 1.27)) hide)
     )
-    (property "MANUFACTURER" "YAEGO" (id 6) (at 49.53 71.12 0)
+    (property "MANUFACTURER" "UNI-ROYAL" (id 6) (at 49.53 71.12 0)
       (effects (font (size 1.27 1.27)) hide)
     )
@@
       (effects (font (size 1.27 1.27)) hide)
     )
-    (property "JLCPCB_PN" "C105588" (id 8) (at 49.53 71.12 0)
+    (property "JLCPCB_PN" "C22775" (id 8) (at 49.53 71.12 0)
       (effects (font (size 1.27 1.27)) hide)
     )
@@
       (effects (font (size 1.27 1.27)) hide)
     )
-    (property "MPN" "RC0603FR-073K3L" (id 4) (at 63.5 74.93 0)
+    (property "MPN" "0603WAF3301T5E" (id 4) (at 63.5 74.93 0)
       (effects (font (size 1.27 1.27)) hide)
     )
@@
       (effects (font (size 1.27 1.27)) hide)
     )
-    (property "MANUFACTURER" "YAEGO" (id 6) (at 63.5 74.93 0)
+    (property "MANUFACTURER" "UNI-ROYAL" (id 6) (at 63.5 74.93 0)
       (effects (font (size 1.27 1.27)) hide)
     )
@@
       (effects (font (size 1.27 1.27)) hide)
     )
-    (property "JLCPCB_PN" "C108078" (id 8) (at 63.5 74.93 0)
+    (property "JLCPCB_PN" "C22978" (id 8) (at 63.5 74.93 0)
       (effects (font (size 1.27 1.27)) hide)
     )
